File: electronic_design/ethersweep/ethersweep.kicad_pcb (KiCad board)
At the start: 2 copper layers, 79 x 38 mm, 101 parts, among them J1 AVR-ISP-6, J10 HR911105A, J11 Conn_01x04_Male, J2 Conn_01x02_Male, J3 Conn_01x04_Female, J4 Conn_01x02_Male, J5 Conn_01x02_Male, J6 Conn_01x07_Female, J7 Conn_01x07_Male, J8 AVR-ISP-6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

Commit message: minor changes
Other:
- board text added: "2022-10-05"
- board text added: "rev. 3.0.5"
- board text removed: "2022-02-22"
- board text removed: "rev. 3.0.4"
Changed lines of the file:
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@@
     (effects (font (size 1 1) (thickness 0.25)) (justify left mirror))
   )
-  (gr_text "rev.\n3.0.4" (at 211.95 61.27) (layer "B.SilkS")
+  (gr_text "rev.\n3.0.5\n" (at 211.95 61.27) (layer "B.SilkS")
     (effects (font (size 1 1) (thickness 0.2)) (justify mirror))
   )
@@
     (effects (font (size 1 1) (thickness 0.25)) (justify mirror))
   )
-  (gr_text "2022-02-22" (at 216.85 58.87) (layer "B.SilkS")
+  (gr_text "2022-10-05" (at 216.85 58.87) (layer "B.SilkS")
     (effects (font (size 1 1) (thickness 0.25)) (justify left mirror))
   )
