File: electronic_design/development/ethersweep406/ethersweep.kicad_pcb (KiCad board)
At the start: 4 copper layers, 79 x 38 mm, 110 parts, among them J1 AVR-ISP-6, J10 HR911105A, J11 USB_B_Micro, J2 Conn_01x02_Male, J3 Conn_01x04_Female, J4 Conn_01x03_Male, J5 Conn_01x03_Male, J6 Conn_01x07_Female, J7 Conn_01x07_Male, J8 AVR-ISP-6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

Commit message: cleanup and minor design changes in 406
Parts:
- added SW2: SW_BOOT_0, Button_Switch_SMD:SW_SPST_B3U-3000P, F.Cu at (188.8, 55.4)
- J11: footprint Connector_USB:USB_Micro-B_Molex_47346-0001 -> Connector_USB:USB_Micro-AB_Molex_47590-0001
- SW1: footprint Button_Switch_SMD:SW_Push_SPST_NO_Alps_SKRK -> Button_Switch_SMD:SW_SPST_B3U-3000P; moved to F.Cu
- moved SW1 32.2 mm to (144.1, 54.7), turned to 90 degrees
- moved J11 0.80 mm to (199.3, 63.3)
Routing:
- net BOOT_0: track 10.7 -> 23.7 mm, vias 1 -> 2
- net rst: track 49.4 -> 43.2 mm
- net Net-(J11-D-): track 4.48 -> 2.30 mm, vias 2 -> 0
- net Net-(J11-VBUS): track 11.3 -> 9.38 mm
- net unconnected-(J11-Shield-Pad6): track 12.6 -> 14.6 mm
- net GND: track 109.5 -> 108.5 mm, vias 78 -> 76
- net +3V3: track 65.6 -> 66.4 mm, vias 20 -> 21
- net SCL: track 99.0 -> 98.2 mm
- net SDA: track 99.4 -> 98.8 mm
Other:
- board text added: "ETHERSWEEP MOTION CONTROLLER 2023-08-17 rev. 4.6.0 github.com/neumi/ethersweep"
- board text added: "v4.6.0"
- board text removed: "ETHERSWEEP MOTION CONTROLLER 2023-05-24 rev. 4.5.0 github.com/neumi/ethersweep"
- board text removed: "v4.5.0"
