File: electronic_design/development/ethersweep406/ethersweep.kicad_sch (KiCad schematic)
At the start: 110 parts, among them J1 AVR-ISP-6, J10 HR911105A, J11 USB_B_Micro, J2 Conn_01x02_Male, J3 Conn_01x04_Female, J4 Conn_01x03_Male, J5 Conn_01x03_Male, J6 Conn_01x07_Female, J7 Conn_01x07_Male, J8 AVR-ISP-6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

Commit message: cleanup and minor design changes in 406
Parts:
- J11: footprint Connector_USB:USB_Micro-B_Molex_47346-0001 -> Connector_USB:USB_Micro-AB_Molex_47590-0001; LCSC C132560 -> C136001
- SW1: footprint Button_Switch_SMD:SW_Push_SPST_NO_Alps_SKRK -> Button_Switch_SMD:SW_SPST_B3U-3000P; LCSC C720477 -> C963349
Changed lines of the file:
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@@
       (effects (font (size 1.27 1.27)))
     )
-    (property "Footprint" "Button_Switch_SMD:SW_Push_SPST_NO_Alps_SKRK" (at 185.674 240.03 0)
+    (property "Footprint" "Button_Switch_SMD:SW_SPST_B3U-3000P" (at 185.674 240.03 0)
       (effects (font (size 1.27 1.27)) hide)
     )
@@
       (effects (font (size 1.27 1.27)) hide)
     )
-    (property "LCSC" "C720477" (at 185.674 245.11 0)
+    (property "LCSC" "C963349" (at 185.674 245.11 0)
       (effects (font (size 1.27 1.27)) hide)
     )
@@
       (effects (font (size 1.27 1.27)) (justify left))
     )
-    (property "Footprint" "Connector_USB:USB_Micro-B_Molex_47346-0001" (at 403.86 211.836 0)
+    (property "Footprint" "Connector_USB:USB_Micro-AB_Molex_47590-0001" (at 403.86 211.836 0)
       (effects (font (size 1.27 1.27)) hide)
     )
@@
       (effects (font (size 1.27 1.27)) hide)
     )
-    (property "LCSC" "C132560" (at 400.05 210.566 0)
+    (property "LCSC" "C136001" (at 400.05 210.566 0)
       (effects (font (size 1.27 1.27)) hide)
     )
